File: TashTalkUSB/TashTalkUSB.kicad_pcb (KiCad board)
At the start: 2 copper layers, 60 x 25 mm, 35 parts, among them J1 TC2030, J3 USB_C_Receptacle_USB2.0_14P, U1 CP2102N-Axx-xQFN20, U2 PIC12F1840-xSN, U3 SN65HVD1473DGSR

Commit message: TashTalkUSB: Final rev 2
Other:
- board text added: "Feral Firmware"
